File: Example/KiCAD_source/Filter DualOp.kicad_pcb (KiCad board)
At the start: 2 copper layers, 33 x 29.2 mm, 13 parts, among them U1 LM4562, U2 LM4562

Commit message: updated KiCAD project files
Parts:
- added ?: , , F.Cu at (131.4, 95.8)
Routing:
- net -5V: track 40.8 -> 43.5 mm
Changed lines of the file:
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@@
     )
+  )
+  (footprint "" (layer "F.Cu")
+    (at 131.360244 95.758)
+    (fp_text reference "" (at 0 0) (layer "F.SilkS")
+      (effects (font (size 1.27 1.27) (thickness 0.15)))
+    )
+    (fp_text value "" (at 0 0) (layer "F.SilkS")
+      (effects (font (size 1.27 1.27) (thickness 0.15)))
+    )
+    (pad "4" thru_hole oval (at 0.1 0.152244) (size 1.6 1.6) (drill 0.8) (layers *.Cu "F.Mask")
+      (net 12 "-5V") (pinfunction "V-") (pintype "power_in"))
   )
   (footprint "Package_DIP:DIP-8_W7.62mm" (layer "F.Cu")
@@
   (segment (start 141.610244 74.300244) (end 138.951204 71.641204) (width 0.5) (layer "F.Cu") (net 12))
   (segment (start 135.280244 95.910244) (end 136.550244 95.910244) (width 0.5) (layer "F.Cu") (net 12))
+  (segment (start 133.35 94.020488) (end 133.35 93.98) (width 0.5) (layer "F.Cu") (net 12))
   (segment (start 132.903667 71.641205) (end 127.521204 77.023668) (width 0.5) (layer "F.Cu") (net 12))
-  (segment (start 127.521204 88.151204) (end 135.280244 95.910244) (width 0.5) (layer "F.Cu") (net 12))
+  (segment (start 133.35 93.98) (end 135.280244 95.910244) (width 0.5) (layer "F.Cu") (net 12))
+  (segment (start 131.460244 95.910244) (end 133.35 94.020488) (width 0.5) (layer "F.Cu") (net 12))
+  (segment (start 127.521204 88.151204) (end 133.35 93.98) (width 0.5) (layer "F.Cu") (net 12))
   (segment (start 133.990244 81.920244) (end 137.800244 81.920244) (width 0.5) (layer "F.Cu") (net 13))
   (segment (start 133.990244 81.920244) (end 131.470244 81.920244) (width 0.5) (layer "F.Cu") (net 13))
